File: Plate Attempt/Bonsai Plate.kicad_pcb (KiCad board)
At the start: 2 copper layers, 348.5 x 137.3 mm, 86 parts

Commit message: Fixed the plate to match the pcb adjustment and cleaned up some of the double lines.
Parts:
- removed SW_LSPC1: SW_Push, MX_Only:MXOnly-2.25U-ReversedStabilizers-NoLED
- moved SW_D1 7.30 mm to (125.4, 143.4)
- moved SW_W1 7.30 mm to (106.0, 119.8)
- moved SW_DASH1 7.30 mm to (279.4, 98.3)
- moved SW_FN1 7.30 mm to (173.1, 192.5)
- moved SW_RGHT1 7.30 mm to (372.1, 180.5)
- moved SW_Y1 7.30 mm to (197.1, 133.0)
- moved SW_K1 7.30 mm to (242.1, 142.9)
- moved SW_A1 7.30 mm to (86.3, 138.5)
- moved SW_E1 7.30 mm to (124.7, 123.7)
- moved SW_R1 7.30 mm to (143.3, 127.7)
- moved SW_[1 7.30 mm to (293.1, 119.5)
- moved SW_APST1 7.30 mm to (302.1, 138.5)
- moved SW_BKSP11 7.30 mm to (317.5, 100.4)
- moved SW_BKSP12 7.30 mm to (336.5, 100.4)
- moved SW_F13 7.30 mm to (144.0, 147.3)
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Other:
- outline, holes or cut-outs redrawn

Commit message: Fixed plate, added art to the PCB and made a base plate with art.
Parts:
- removed SW_BKSP1: SW_Push, MX_Only:MXOnly-2U-NoLED
- removed SW_BKSP11, SW_BKSP12, SW_FN1: SW_Push, MX_Only:MXOnly-1U-NoLED
- removed SW_CPLK1: SW_Push, MX_Only:MXOnly-1.75U-NoLED
- removed SW_CPLKSTPD1, SW_FN2: SW_Push, MX_Only:MXOnly-1.25U-NoLED
- moved SW_F11 9.21 mm to (295.6, 84.8)
- moved SW_COMMA1 9.21 mm to (251.5, 167.2)
- moved SW_UP1 9.21 mm to (348.2, 169.3)
- moved SW_TAB1 9.21 mm to (57.0, 127.3)
- moved SW_1 9.21 mm to (75.4, 108.3)
- moved SW_ENT1 9.21 mm to (328.3, 146.4)
- moved SW_F13 9.21 mm to (139.2, 155.2)
- moved SW_F2 9.21 mm to (79.0, 84.8)
- moved SW_K1 9.21 mm to (237.3, 150.8)
- moved SW_M3 9.21 mm to (363.0, 127.2)
- moved SW_SLSH1 9.21 mm to (292.0, 165.4)
- moved SW_10 9.21 mm to (253.6, 108.4)
- moved SW_6 9.21 mm to (170.4, 122.9)
- moved SW_9 9.21 mm to (235.0, 112.3)
- moved SW_LALT1 9.21 mm to (102.9, 187.2)
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Other:
- outline, holes or cut-outs redrawn
