File: Bonsai.kicad_pcb (KiCad board)
At the start: 2 copper layers, 348.5 x 165.6 mm, 204 parts, among them J1 AVR-ISP-6, U1 ATmega32A-PU, Y1 Crystal

Commit message: Removed the hole labels from the silk screen.
Parts:
- C5: footprint cftkb:D_DO-35_SOD27_P5.08mm_Horizontal -> cftkb:C_Disc_D4.3mm_W1.9mm_P5.00mm
- moved C5 1.12 mm to (178.7, 81.4)
