File: Base Plate/Bonsai Base Plate/Bonsai Base Plate.kicad_pcb (KiCad board)
At the start: 2 copper layers, 348.5 x 165.6 mm, 13 parts

Commit message: Removed the hole labels from the silk screen.
Routing:
- net (no net): track 30.5 -> 0.00 mm
Changed lines of the file:
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@@
     (thickness 1.6)
     (drawings 12)
-    (tracks 1)
+    (tracks 0)
     (zones 0)
     (modules 13)
@@
     (tags "mounting hole 2.2mm no annular m2")
     (attr virtual)
-    (fp_text reference H12 (at 0 -3.2) (layer F.SilkS)
+    (fp_text reference H12 (at 0 -3.2) (layer F.SilkS) hide
       (effects (font (size 1 1) (thickness 0.15)))
     )
@@
     (tags "mounting hole 2.2mm no annular m2")
     (attr virtual)
-    (fp_text reference H11 (at 0 -3.2) (layer F.SilkS)
+    (fp_text reference H11 (at 0 -3.2) (layer F.SilkS) hide
       (effects (font (size 1 1) (thickness 0.15)))
     )
@@
     (tags "mounting hole 2.2mm no annular m2")
     (attr virtual)
-    (fp_text reference H10 (at 0 -3.2) (layer F.SilkS)
+    (fp_text reference H10 (at 0 -3.2) (layer F.SilkS) hide
       (effects (font (size 1 1) (thickness 0.15)))
     )
@@
     (tags "mounting hole 2.2mm no annular m2")
     (attr virtual)
-    (fp_text reference H9 (at 0 -3.2) (layer F.SilkS)
+    (fp_text reference H9 (at 0 -3.2) (layer F.SilkS) hide
       (effects (font (size 1 1) (thickness 0.15)))
     )
@@
     (tags "mounting hole 2.2mm no annular m2")
     (attr virtual)
-    (fp_text reference H8 (at 0 -3.2) (layer F.SilkS)
+    (fp_text reference H8 (at 0 -3.2) (layer F.SilkS) hide
       (effects (font (size 1 1) (thickness 0.15)))
     )
@@
     (tags "mounting hole 2.2mm no annular m2")
     (attr virtual)
-    (fp_text reference H7 (at 0 -3.2) (layer F.SilkS)
+    (fp_text reference H7 (at 0 -3.2) (layer F.SilkS) hide
       (effects (font (size 1 1) (thickness 0.15)))
     )
@@
     (tags "mounting hole 2.2mm no annular m2")
     (attr virtual)
-    (fp_text reference H6 (at 0 -3.2) (layer F.SilkS)
+    (fp_text reference H6 (at 0 -3.2) (layer F.SilkS) hide
       (effects (font (size 1 1) (thickness 0.15)))
     )
@@
     (tags "mounting hole 2.2mm no annular m2")
     (attr virtual)
-    (fp_text reference H5 (at 0 -3.2) (layer F.SilkS)
+    (fp_text reference H5 (at 0 -3.2) (layer F.SilkS) hide
       (effects (font (size 1 1) (thickness 0.15)))
     )
@@
     (tags "mounting hole 2.2mm no annular m2")
     (attr virtual)
-    (fp_text reference H4 (at 0 -3.2) (layer F.SilkS)
+    (fp_text reference H4 (at 0 -3.2) (layer F.SilkS) hide
       (effects (font (size 1 1) (thickness 0.15)))
     )
@@
     (tags "mounting hole 2.2mm no annular m2")
     (attr virtual)
-    (fp_text reference H3 (at 0 -3.2) (layer F.SilkS)
+    (fp_text reference H3 (at 0 -3.2) (layer F.SilkS) hide
       (effects (font (size 1 1) (thickness 0.15)))
     )
@@
     (tags "mounting hole 2.2mm no annular m2")
     (attr virtual)
-    (fp_text reference H2 (at 0 -3.2) (layer F.SilkS)
+    (fp_text reference H2 (at 0 -3.2) (layer F.SilkS) hide
       (effects (font (size 1 1) (thickness 0.15)))
     )
@@
     (tags "mounting hole 2.2mm no annular m2")
     (attr virtual)
-    (fp_text reference H1 (at 0 -3.2) (layer F.SilkS)
+    (fp_text reference H1 (at 0 -3.2) (layer F.SilkS) hide
       (effects (font (size 1 1) (thickness 0.15)))
     )
@@
   (gr_arc (start 379.903991 63.08725) (end 384.70205 63.04915) (angle -90) (layer Edge.Cuts) (width 0.05))
   (gr_arc (start 379.901452 205.474571) (end 379.89129 210.27263) (angle -90) (layer Edge.Cuts) (width 0.05))
-  (segment (start 298.354026 58.932609) (end 267.86428 58.932609) (width 0.254) (layer F.Cu) (net 0))
 )
